Commit message: Gazebo model of M10iA is working

File: src/fanuc_description/urdf/m10ia_macro.xacro (robot description, xacro)
@@ -8,5 +8,5 @@
         <origin xyz="0 0 0" rpy="0 0 0"/>
         <geometry>
-          <mesh filename="package://fanuc_description/meshes/m10ia/visual/base_link.stl"/>
+          <mesh filename="package://fanuc_description/meshes/m10ia/visual/base_link.stl" scale="0.001 0.001 0.001"/>
         </geometry>
         <xacro:material_fanuc_gray40 />
@@ -15,5 +15,5 @@
         <origin xyz="0 0 0" rpy="0 0 0"/>
         <geometry>
-          <mesh filename="package://fanuc_description/meshes/m10ia/collision/base_link.stl"/>
+          <mesh filename="package://fanuc_description/meshes/m10ia/collision/base_link.stl" scale="0.001 0.001 0.001"/>
         </geometry>
       </collision>
@@ -23,5 +23,5 @@
         <origin xyz="0 0 0" rpy="0 0 0"/>
         <geometry>
-          <mesh filename="package://fanuc_description/meshes/m10ia/visual/link_1.stl"/>
+          <mesh filename="package://fanuc_description/meshes/m10ia/visual/link_1.stl" scale="0.001 0.001 0.001"/>
         </geometry>
         <xacro:material_fanuc_yellow />
@@ -30,5 +30,5 @@
         <origin xyz="0 0 0" rpy="0 0 0"/>
         <geometry>
-          <mesh filename="package://fanuc_description/meshes/m10ia/collision/link_1.stl"/>
+          <mesh filename="package://fanuc_description/meshes/m10ia/collision/link_1.stl" scale="0.001 0.001 0.001"/>
         </geometry>
       </collision>
@@ -38,5 +38,5 @@
         <origin xyz="0 0 0" rpy="0 0 0"/>
         <geometry>
-          <mesh filename="package://fanuc_description/meshes/m10ia/visual/link_2.stl"/>
+          <mesh filename="package://fanuc_description/meshes/m10ia/visual/link_2.stl" scale="0.001 0.001 0.001"/>
         </geometry>
         <xacro:material_fanuc_yellow />
@@ -45,5 +45,5 @@
         <origin xyz="0 0 0" rpy="0 0 0"/>
         <geometry>
-          <mesh filename="package://fanuc_description/meshes/m10ia/collision/link_2.stl"/>
+          <mesh filename="package://fanuc_description/meshes/m10ia/collision/link_2.stl" scale="0.001 0.001 0.001"/>
         </geometry>
       </collision>
@@ -53,5 +53,5 @@
         <origin xyz="0 0 0" rpy="0 0 0"/>
         <geometry>
-          <mesh filename="package://fanuc_description/meshes/m10ia/visual/link_3.stl"/>
+          <mesh filename="package://fanuc_description/meshes/m10ia/visual/link_3.stl" scale="0.001 0.001 0.001"/>
         </geometry>
         <xacro:material_fanuc_yellow />
@@ -60,5 +60,5 @@
         <origin xyz="0 0 0" rpy="0 0 0"/>
         <geometry>
-          <mesh filename="package://fanuc_description/meshes/m10ia/collision/link_3.stl"/>
+          <mesh filename="package://fanuc_description/meshes/m10ia/collision/link_3.stl" scale="0.001 0.001 0.001"/>
         </geometry>
       </collision>
@@ -68,5 +68,5 @@
         <origin xyz="0 0 0" rpy="0 0 0"/>
         <geometry>
-          <mesh filename="package://fanuc_description/meshes/m10ia/visual/link_4.stl"/>
+          <mesh filename="package://fanuc_description/meshes/m10ia/visual/link_4.stl" scale="0.001 0.001 0.001"/>
         </geometry>
         <xacro:material_fanuc_yellow />
@@ -75,5 +75,5 @@
         <origin xyz="0 0 0" rpy="0 0 0"/>
         <geometry>
-          <mesh filename="package://fanuc_description/meshes/m10ia/collision/link_4.stl"/>
+          <mesh filename="package://fanuc_description/meshes/m10ia/collision/link_4.stl" scale="0.001 0.001 0.001"/>
         </geometry>
       </collision>
@@ -83,5 +83,5 @@
         <origin xyz="0 0 0" rpy="0 0 0"/>
         <geometry>
-          <mesh filename="package://fanuc_description/meshes/m10ia/visual/link_5.stl"/>
+          <mesh filename="package://fanuc_description/meshes/m10ia/visual/link_5.stl" scale="0.001 0.001 0.001"/>
         </geometry>
         <xacro:material_fanuc_yellow />
@@ -90,5 +90,5 @@
         <origin xyz="0 0 0" rpy="0 0 0"/>
         <geometry>
-          <mesh filename="package://fanuc_description/meshes/m10ia/collision/link_5.stl"/>
+          <mesh filename="package://fanuc_description/meshes/m10ia/collision/link_5.stl" scale="0.001 0.001 0.001"/>
         </geometry>
       </collision>
@@ -98,5 +98,5 @@
         <origin xyz="0 0 0" rpy="0 0 0"/>
         <geometry>
-          <mesh filename="package://fanuc_description/meshes/m10ia/visual/link_6.stl"/>
+          <mesh filename="package://fanuc_description/meshes/m10ia/visual/link_6.stl" scale="0.001 0.001 0.001"/>
         </geometry>
         <xacro:material_fanuc_black />
@@ -105,5 +105,5 @@
         <origin xyz="0 0 0" rpy="0 0 0"/>
         <geometry>
-          <mesh filename="package://fanuc_description/meshes/m10ia/collision/link_6.stl"/>
+          <mesh filename="package://fanuc_description/meshes/m10ia/collision/link_6.stl" scale="0.001 0.001 0.001"/>
         </geometry>
       </collision>
@@ -146,5 +146,5 @@
     </joint>
     <joint name="${prefix}joint_6" type="revolute">
-      <origin xyz="0.100 0 0" rpy="0 0 0"/>
+      <origin xyz="0 0 0" rpy="0 0 0"/>
       <parent link="${prefix}link_5"/>
       <child link="${prefix}link_6"/>
@@ -162,5 +162,5 @@
     <link name="${prefix}flange" />
     <joint name="${prefix}joint_6-flange" type="fixed">
-      <origin xyz="0 0 0" rpy="0 0 0" />
+      <origin xyz="0.1 0 0" rpy="0 0 0" />
       <parent link="${prefix}link_6" />
       <child link="${prefix}flange" />
@@ -169,5 +169,5 @@
     <link name="${prefix}tool0" />
     <joint name="${prefix}link_6-tool0" type="fixed">
-      <origin xyz="0 0 0" rpy="${pi} ${-pi/2.0} 0" />
+      <origin xyz="0.1 0 0" rpy="${pi} ${-pi/2.0} 0" />
       <parent link="${prefix}flange" />
       <child link="${prefix}tool0" />
